File: cad/IceCore.brd (EAGLE design)
At the start: 50 x 50 mm, 131 parts, among them IC1 ICE40HX4K_TQFP144, IC2 STM32F103RET6, IC3 SDRAM, X100 1296-T50, X101 1296-T50, Y1 12MZ

Commit message: Updated Readme
Parts:
- moved SD100 0.82 mm to (42.5, 15.5)
Routing:
- net A2: track 33.7 -> 36.4 mm
- net +3V3: track 123.2 -> 121.1 mm, vias 28 -> 29
- net SDCLK: track 34.2 -> 36.0 mm
- net A6: track 21.1 -> 22.3 mm
- net SD0: track 33.1 -> 33.9 mm
- net L0: track 60.8 -> 61.6 mm
- net SD1: track 33.4 -> 34.2 mm
- net SD2: track 35.7 -> 36.4 mm
- net GND: track 6.55 -> 6.66 mm, vias 60 -> 61
Other:
- board text added: "F1"
- board text added: "U$11"
- board text added: "U$3"
- board text added: "U$4"
- board text added: "U$5"
- board text added: "U$6"
- board text added: "U$7"
- board text added: "V1.2-HX40-4/16Mb 22 May 2019"
- board text added: "Y1"
- board text removed: "V1.2-HX40-4/16Mb Week 18 May 2019"
